Commit message: add controll but is wrong it need fix

File: src/manipulation_description/urdf/arm.xacro (robot description, xacro)
@@ -1,4 +1,13 @@
 <?xml version="1.0"?>
 <robot xmlns:xacro="http://www.ros.org/wiki/xacro">
+    <xacro:macro name="default_transmission" params="number">
+        <transmission name="transmission_${number}">
+            <plugin>transmission_interface/SimpleTransmission</plugin>
+            <actuator name="motor_${number}" role="actuator1" />
+            <joint name="axis${number}_joint" role="joint1">
+                <mechanical_reduction>1.0</mechanical_reduction>
+            </joint>
+        </transmission>
+    </xacro:macro>
     <link name="base_footprint" />
     <link name="arm_base_link">
@@ -488,3 +497,9 @@
         <dynamics friction="0.05" damping="0.1"/>
     </joint>
+    <xacro:default_transmission number="1"/>
+    <xacro:default_transmission number="2"/>
+    <xacro:default_transmission number="3"/>
+    <xacro:default_transmission number="4"/>
+    <xacro:default_transmission number="5"/>
+    <xacro:default_transmission number="6"/>
 </robot>

File: src/manipulation_description/urdf/arm_gazebo.xacro (robot description, xacro)
@@ -1,4 +1,11 @@
 <?xml version="1.0"?>
-<robot xmlns:xacro="http://www.ros.org/wiki/xacro">
+<robot xmlns:xacro="http://www.ros.org/wiki/xacro" name="manipulation">
+    <gazebo>
+        <plugin filename="libgazebo_ros2_control.so" name="gazebo_ros2_control">
+            <robot_param>robot_description</robot_param>
+            <robot_param_node>robot_state_publisher</robot_param_node>
+            <parameters>$(find manipulation_controller)/config/manipulation_controllers.yaml</parameters>
+        </plugin>
+    </gazebo>
     <gazebo reference="arm_base_link">
         <material>Gazebo/Grey</material>
@@ -43,24 +50,3 @@
         <material>Gazebo/Red</material>
     </gazebo>
-    <gazebo>
-        <plugin name="joint_state_publisher_controller"
-                filename="libgazebo_ros_joint_state_publisher.so">
-            <!-- Update rate in Hertz -->
-            <update_rate>10</update_rate>
-            <!-- Name of joints in the model whose states will be published. -->
-            <joint_name>axis1_joint</joint_name>
-            <joint_name>axis2_joint</joint_name>
-            <joint_name>axis3_joint</joint_name>
-            <joint_name>axis4_joint</joint_name>
-            <joint_name>axis5_joint</joint_name>
-            <joint_name>axis6_joint</joint_name>
-        </plugin>
-    </gazebo>
-    <gazebo>
-        <plugin name="joint_pose_trajectory_controller"
-                filename="libgazebo_ros_joint_pose_trajectory.so">
-            <!-- Update rate in Hz -->
-            <update_rate>2</update_rate>
-        </plugin>
-    </gazebo>
 </robot>

File: src/manipulation_description/urdf/manipulation.urdf.xacro (robot description, xacro)
@@ -4,3 +4,4 @@
     <xacro:include filename="arm.xacro" />
     <xacro:include filename="arm_gazebo.xacro" />
+    <xacro:include filename="arm_ros2_control.xacro" />
 </robot>
